Commit message: Created Gazebo world to navigate in

File: description/robot_core.xacro (robot description, xacro)
@@ -41,4 +41,7 @@
         </xacro:inertial_box>
     </link>
+    <gazebo reference="chassis">
+        <material>Gazebo/White</material>
+    </gazebo>
     <!--LEFT WHEEL -->
     <joint name="left_wheel_joint" type="continuous">
@@ -64,4 +67,7 @@
         </xacro:inertial_cylinder>
     </link>
+    <gazebo reference="left_wheel">
+        <material>Gazebo/Blue</material>
+    </gazebo>
     <!--RIGHT WHEEL -->
     <joint name="right_wheel_joint" type="continuous">
@@ -87,4 +93,7 @@
         </xacro:inertial_cylinder>
     </link>
+    <gazebo reference="right_wheel">
+        <material>Gazebo/Blue</material>
+    </gazebo>
     <!-- Left Castor Wheel -->
     <joint name="left_castor_wheel_joint" type="fixed">
@@ -110,4 +119,9 @@
         </xacro:inertial_cylinder>
     </link>
+    <gazebo reference="left_castor_wheel">
+        <material>Gazebo/Black</material>
+        <mu1 value="0.001"/>
+        <mu2 value="0.001"/>
+    </gazebo>
     <!-- Right Castor Wheel -->
     <joint name="right_castor_wheel_joint" type="fixed">
@@ -133,3 +147,8 @@
         </xacro:inertial_cylinder>
     </link>
+    <gazebo reference="right_castor_wheel">
+        <material>Gazebo/Black</material>
+        <mu1 value="0.001"/>
+        <mu2 value="0.001"/>
+    </gazebo>
 </robot>

Commit message: SLAM implementation - final touches

File: description/robot_core.xacro (robot description, xacro)
@@ -68,5 +68,5 @@
         <collision>
             <geometry>
-                <cylinder radius="0.0625" length="0.0775"/>
+                <sphere radius="0.0625"/>
             </geometry>
         </collision>
@@ -94,5 +94,5 @@
         <collision>
             <geometry>
-                <cylinder radius="0.0625" length="0.0775"/>
+                <sphere radius="0.0625"/>
             </geometry>
         </collision>
